Commit message: fix: solve nan output of nn-based policy
- use obs checking/reverting and grad clipping to avoid nan
- update dubins car urdf (kobuki, sensors)
- add angle as part of goal of car env
- test several action transformation in step()
- add scatter plotter for showing result
- minor code refactor

File: urdfs/kobuki_nn_urdf/urdf/kobuki.urdf.xacro (robot description, xacro)
@@ -6,9 +6,9 @@
       kobuki_description/launch/view_model.launch
  -->
-<robot xmlns:xacro="http://ros.org/wiki/xacro">
-  <!--<xacro:include filename="$(find kobuki_description)/urdf/common_properties.urdf.xacro"/>-->
-  <!--<xacro:include filename="$(find kobuki_description)/urdf/kobuki_gazebo.urdf.xacro"/>-->
+<robot name="kobuki" xmlns:xacro="http://ros.org/wiki/xacro">
+  <xacro:include filename="$(find kobuki_description)/urdf/common_properties.urdf.xacro"/>
+  <xacro:include filename="$(find kobuki_description)/urdf/kobuki_gazebo.urdf.xacro"/>
   <!-- Kobuki -->
-  <xacro:macro name="dubins_car_base_macro">
+  <xacro:macro name="kobuki">
     <link name="base_footprint"/>
     <!--
@@ -208,6 +208,6 @@
       </inertial>
     </link>
-    <!--&lt;!&ndash; Kobuki Gazebo simulation details &ndash;&gt;-->
-    <!--<kobuki_sim/>-->
+    <!-- Kobuki Gazebo simulation details -->
+    <kobuki_sim/>
   </xacro:macro>
   <!-- Lidar sensor -->
@@ -222,13 +222,8 @@
     field_of_view_horizontal="${270*M_PI/180}"
     field_of_view_vertical="${1*M_PI/180}"
-    ray_count_horizontal="40"
+    ray_count_horizontal="200"
     ray_count_vertical="1"
     sensor_mesh="lidar_lite_v2_withRay/meshes/lidar_lite_v2_withRay.dae">
     <origin xyz="0 0.0 0.5" rpy="0 0 0"/>
   </xacro:lidar_sensor>
-    <!-- hexagon stack -->
-    <xacro:include filename="$(find turtlebot_description)/urdf/stacks/hexagons.urdf.xacro"/>
-    <xacro:stack_hexagons
-            parent="base_link">
-    </xacro:stack_hexagons>>
 </robot>
